File: pcb/claudepad_render.kicad_pcb (KiCad board)
At the start: 2 copper layers, 98 x 50 mm, 35 parts, among them SW1 ChocV2, SW10 ChocV2, SW11 ChocV2, SW12 ChocV2, SW13 ChocV2, SW14 ChocV2, SW2 ChocV2, SW3 ChocV2, SW4 ChocV2, SW5 ChocV2, SW6 ChocV2, SW7 ChocV2, SW8 ChocV2, SW9 ChocV2

Commit message: 布局再改：空格那行 4 颗键贴左排（跨列 1-3 + 语音列 4）+ 定位板切孔 bug 修复
用户原话（2026-10-11）：'最下层不是有四个键而已吗？我们之间给他并排与上方对其'
+ 澄清 '第 1~4 列，最左列不该空出来'。上一版误改成跨列 2-4 + 最左列空出，方向反了。

【1】空格行贴左
  KEYMAP [2,3,3,SPACE] + [5,3,1,VOICE] → [1,3,3,SPACE] + [4,3,1,VOICE]
  空格 3 轴 31/49/67 → 13/31/49（全部落在 18mm 网格线上）；语音键列 5 → 列 4
  列 5（x=85）空出 → 主控上方不再压任何轴体（原 VOICE 正好压在主控上）
  连带：overlay 矩阵变换末行 RC(2,4) → RC(2,3)；空格 net COL2 → COL1

【2】★ 定位板切孔 bug（渲染预览时发现）
  choc_cutout() 用 linear_extrude(center=true) 又被 translate z=-1，
  切槽只覆盖 z[-2.6,0.6]，而板厚 [0,1.2] → 顶面留 0.6mm 皮没切穿。
  STL 体积 6.33 cm³（实心板 + 4 螺丝孔）→ 修后 4.61 cm³。
  也就是说：**之前导出的定位板 STL 轴体根本插不进去**。

【3】展示层修漂移（都是会撒谎的硬拷贝）
  · tools/render_assembly.py：写死的板宽 98 / JP 80.97 / NANO 79.70 / 空格 31-49-67
    → 全改为读 pcb/placement.csv + 板文件 + params；俯视图孔位改为按真实旋转角算
    （原先只做 180° 镜像，STOP 270° / ENTER 90° 的孔画错位置）
  · cad/pcb_assembly.scad：SWITCHES / JP_XS / JP_N / 主控位置与 USB 朝向 / 复位焊盘
  · tools/check_dims.py：空格挠度按 4u 算 → 从 KEYMAP 推导（3u：单轴 0.67 / 三轴 0.08）
  · 新增 tools/render_board_annotated.py：board-annotated.png 等改由脚本生成

【4】重生成产物
  pcb/claudepad.kicad_pcb（99×50）· pcb/steps/*（6 个）· placement.csv / netlist / wiring
  cad/output/*.stl（6 个，含修好的定位板）· docs/img/*（板子 5 视角 + 分步 8 张 +
  焊接参考图 + 标注图 + 顶视预览）· pcb/claudepad_render.kicad_pcb（含 3D 模型）

【5】文档同步：焊接指南 / PCB 规格书 / 打样下单指南 / 改板方案 / PRD / 结构 / 采购 /
  项目报告 / README / firmware README / MEMORY.md（4u→3u、98→99、排针列位、主控坐标）

校验：check_dims 29/29 · lint_scad · verify_geometry · check_keymap · verify_stl ·
test_hook 全过；DRC 0 错误（39 条丝印警告 + 59 未连接，未布线预期）
⚠️ 尚未布线、未出 Gerber（打样前必须补）
Parts:
- JP1, JP2: footprint PinHeader_1x12_P2.54mm_Vertical -> PinHeader_1x13_P2.54mm_Vertical
- moved SW13 18.0 mm to (49.0, 7.00)
- moved SW14 18.0 mm to (67.0, 7.00)
- moved SW12 9.00 mm to (31.0, 7.00)
- moved GND1 5.66 mm to (74.0, 37.0)
- moved JP1 3.75 mm to (78.0, 4.70)
- moved JP2 3.75 mm to (93.3, 4.70)
- moved RGB1 0.50 mm to (75.5, 28.0)
- turned SW10 to 90 degrees
- turned SW5 to -90 degrees
Connections:
- D12 pad 2: COL5 -> COL4
- JP1 pad 1: (no net) -> GND
- JP1 pad 10: COL1 -> ROW3
- JP1 pad 11: COL2 -> COL1
- JP1 pad 12: COL3 -> COL2
- JP1 pad 3: GND -> (no net)
- JP1 pad 5: (no net) -> GND
- JP1 pad 7: ROW1 -> (no net)
- JP1 pad 8: ROW2 -> ROW1
- JP1 pad 9: ROW3 -> ROW2
- JP2 pad 10: COL6 -> RGB_DIN
- JP2 pad 11: COL5 -> COL6
- JP2 pad 12: COL4 -> COL5
- JP2 pad 2: GND -> (no net)
- JP2 pad 3: RST -> GND
- JP2 pad 4: (no net) -> RST
- JP2 pad 9: RGB_DIN -> (no net)
- SW14 pad 1: COL5 -> COL4
Routing:
- net ROW1: track 148.3 -> 0.00 mm
- net COL1: track 142.1 -> 0.00 mm
- net ROW2: track 137.4 -> 0.00 mm
- net ROW3: track 128.4 -> 0.00 mm
- net COL2: track 93.4 -> 0.00 mm
- net COL3: track 91.5 -> 0.00 mm
- net COL4: track 81.8 -> 0.00 mm
- net COL5: track 75.3 -> 0.00 mm
- net GND: track 38.4 -> 0.00 mm
- net RST: track 38.2 -> 0.00 mm, vias 2 -> 0
- net COL6: track 26.8 -> 0.00 mm
- net RGB_DIN: track 20.9 -> 0.00 mm
Other:
- board size 98 x 50 mm -> 99 x 50 mm
- board text added: "USB -> +Y WALL (top)"
- board text removed: "USB -> RIGHT WALL"

Commit message: 布线完成 + 修致命电路拓扑（二极管/轴体并联 → 串联）+ 出 Gerber
⚠️ 用户要求『去嘉立创下单』，但板子当时不能下单：没布线、Gerber 是第一版的。
   本次把前置条件全部做完了。

【1】★ 致命电路错误：二极管与轴体并联（发现于核对焊盘网络）
  SW1: pad1→COL1, pad2→ROW1 ／ D1: K→ROW1, A→COL1 —— 两者**并联**。
  后果：驱动任一列都会经二极管直接灌通行线 → 该列按键恒为『按下』，键盘不可用。
  正解（与 netlist.md 的『列 → 阳极 → 阴极 → 轴体 → 行』一致）是**串联**：
      列 COL ── A▷|── K ── MID ── 轴体pad1 ──[按下]── pad2 ── ROW
  · gen_pcb.py：每个矩阵位置新增局部网络 net_mid（大键多轴共用；拨杆用 APPROVE_MID）
  · gen_kicad.py：轴体 pad1→MID / pad2→ROW；二极管 K→MID / A→COL
  · gen_kicad.py 自检新增**串联断言**（几何检查查不出这类错，必须断言网络）
  · 第一版板子也带这个错（已作废，未流出）

【2】自动布线（打通链路）
  tools/export_dsn.py（新增）→ FreeRouting → tools/import_ses.py → 174 段 + 3 过孔
  · FreeRouting 原生 CLI v2.5.0 在本项目 DSN 上崩（GraalVM 序列化限制），
    改用 freerouting-1.9.0.jar + OpenJDK 21（1.7 秒布完）
  · tools/patch_route.py（新增）补自动布线漏掉的 ROW3 一段（绕开两个 Ø5 中心孔）
  · DRC：**0 错误 / 0 未连接**（39 条丝印警告为既有，不影响打样）

【3】出 Gerber（第二版打样包）
  pcb/fabrication/claudepad-jlc.zip —— 10 个文件（F/B 铜箔·阻焊·丝印 + 板框 + 钻孔 + 网表）
  第一版全套（含 9-28 的 zip）归档到 pcb/fabrication/v1-2026-09-28/，避免误下单

【4】文档
  · 打样下单指南：状态改为『可以下单』，补下单参数（建议勾飞针电测）与到货核对项
  · 焊接指南：二极管极性说明改为串联口径；★ 新增『列 ↔ 行 不导通』万用表检查
  · 全部『阳极接列、阴极接行』措辞改为『阳极朝列、阴极朝行（与轴体串联）』
  · MEMORY.md：新增布线/打样链路一节（含 FreeRouting 版本坑与镜像）

校验：check_dims 29/29 · lint_scad · verify_geometry · check_keymap · verify_stl ·
test_hook 全过；DRC 0 错误 / 0 未连接
Connections:
- D1 pad 1: ROW1 -> MID_R1C1
- D10 pad 1: ROW2 -> MID_R2C4
- D11 pad 1: ROW3 -> MID_R3C1
- D12 pad 1: ROW3 -> MID_R3C4
- D2 pad 1: ROW1 -> MID_R1C2
- D3 pad 1: ROW1 -> MID_R1C3
- D4 pad 1: ROW1 -> MID_R1C4
- D5 pad 1: ROW1 -> MID_R1C5
- D6 pad 1: ROW1 -> APPROVE_MID
- D7 pad 1: ROW2 -> MID_R2C1
- D8 pad 1: ROW2 -> MID_R2C2
- D9 pad 1: ROW2 -> MID_R2C3
- SW1 pad 1: COL1 -> MID_R1C1
- SW10 pad 1: COL4 -> MID_R2C4
- SW11 pad 1: COL1 -> MID_R3C1
- SW12 pad 1: COL1 -> MID_R3C1
- SW13 pad 1: COL1 -> MID_R3C1
- SW14 pad 1: COL4 -> MID_R3C4
- SW2 pad 1: COL2 -> MID_R1C2
- SW3 pad 1: COL3 -> MID_R1C3
- SW4 pad 1: COL4 -> MID_R1C4
- SW5 pad 1: COL5 -> MID_R1C5
- SW6 pad 1: COL1 -> MID_R2C1
- SW7 pad 1: COL2 -> MID_R2C2
- SW8 pad 1: COL3 -> MID_R2C3
- SW9 pad 1: COL4 -> MID_R2C4
Routing:
- net ROW1: track 0.00 -> 111.2 mm, vias 0 -> 1
- net ROW3: track 0.00 -> 102.0 mm
- net COL1: track 0.00 -> 101.0 mm
- net ROW2: track 0.00 -> 91.6 mm
- net COL2: track 0.00 -> 77.4 mm
- net COL3: track 0.00 -> 70.5 mm, vias 0 -> 1
- net COL4: track 0.00 -> 67.0 mm, vias 0 -> 1
- net GND: track 0.00 -> 56.9 mm
- net MID_R3C1: track 0.00 -> 52.1 mm
- net RST: track 0.00 -> 44.5 mm
- net MID_R2C4: track 0.00 -> 40.3 mm
- net MID_R1C5: track 0.00 -> 38.3 mm
- net COL5: track 0.00 -> 34.4 mm
- net APPROVE_MID: track 0.00 -> 30.0 mm
- net MID_R2C3: track 0.00 -> 23.7 mm
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